File: AutonomousWiringKiCad/AutonomousWiring.kicad_sch (KiCad schematic)
At the start: 21 parts

Commit message: Fix names
Parts:
- renumbered EStop1 to EStop, F2 to F1, KartOn1 to KartOn, PreCharge1 to PreCharge, ev_battery2 to ev_battery, ev_bullet1 to ev_bullet, ev_contactor2 to ev_contactor, ev_dcdc_24v1 to ev_dcdc_24v, ev_dcdc_5v2 to ev_dcdc_5v, ev_dcusbcpd2 to ev_dcusbcpd, ev_eth_switch1 to ev_eth_switch, ev_poe_adp1 to ev_poe_adp, ev_rc_reciever2 to ev_rc_reciever, ev_rtk_gps1 to ev_rtk_gps, ev_steering2 to ev_steering, ev_nucleo2 to ev_stm32, ev_vesc2 to ev_vesc
Connections:
- net at ev_stm32. (Mode_PWM): now also ev_vesc. (Phase3)
- net at ev_contactor_nmos2. (Drain): now also ev_contactor_nmos1. (Drain); no longer ev_stm32. (Mode_PWM)
- net at ev_contactor. (Feedback2): now also ev_contactor_nmos1. (Drain); no longer ev_stm32. (Mode_PWM)
- net at ev_rc_reciever. (GND): now also EStop.2 (B), ev_dcdc_5v. (5v); no longer ev_stm32. (Mode_PWM)
- net at ev_rubik1. (GND): now also ev_dcusbcpd. (USB-C_PD); no longer ev_stm32. (Mode_PWM)
- net at ev_poe_adp. (POE_Eth): now also ev_bullet. (PoE_Eth); no longer ev_eth_switch. (ETH6)
- net at ev_contactor_nmos1. (Drain): now also PWM_to_Analog.1; no longer ev_contactor_nmos2. (Drain)
- net at ev_battery. (Contactor2): now also EStop.1 (A); no longer ev_contactor. (Feedback2)
- new net: ev_battery. (Contactor2), ev_contactor_nmos2. (Drain), ev_dcdc_24v. (24v), ev_dcdc_5v. (5v), ev_eth_switch. (ETH6), ev_poe_adp. (POE_Eth), ev_rc_reciever. (GND), ev_steering. (GND), ev_vesc. (Phase3)
- new net: ev_dcdc_24v. (24v), ev_dcdc_5v. (5v), ev_dcusbcpd. (USB-C_PD), ev_eth_switch. (ETH6), ev_poe_adp. (POE_Eth), ev_steering. (GND)
- new net: ev_contactor_nmos2. (Drain), ev_stm32. (Mode_PWM)
- new net: ev_steering. (GND), ev_stm32. (Mode_PWM)
- new net: ev_contactor. (Feedback2), ev_stm32. (Mode_PWM) (x2)
- new net: PWM_to_Analog.2, ev_rc_reciever. (GND), ev_stm32. (Mode_PWM)
- new net: ev_rc_reciever. (GND), ev_stm32. (Mode_PWM) (x3)
- new net: ev_rubik1. (GND), ev_stm32. (Mode_PWM) (x6)
- new net: ev_stm32. (Mode_PWM), ev_vesc. (Phase3) (x2)
- new net: F1.1, ev_battery. (Contactor2), ev_contactor. (Feedback2)
- new net: ev_eth_switch. (ETH6), ev_poe_adp. (POE_Eth)
- new net: ev_battery. (Contactor2), ev_contactor. (Feedback2)
- new net: PreCharge.1, ev_contactor. (Feedback2), ev_vesc. (Phase3)
- new net: ev_eth_switch. (ETH6), ev_rubik1. (GND)
- new net: ev_rtk_gps. (GND), ev_rubik1. (GND) (x3)
Changed lines of the file:
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@@
 		(on_board yes)
 		(dnp no)
-		(property "Reference" "KartOn1"
+		(property "Reference" "KartOn"
 			(at 57.15 35.052 0)
 			(effects
@@
 			(project "AutonomousWiring"
 				(path "/f9355d6c-5335-47ee-824d-8b7223514fe3"
-					(reference "KartOn1")
+					(reference "KartOn")
 					(unit 1)
 				)
@@
 		(on_board yes)
 		(dnp no)
-		(property "Reference" "ev_dcdc_24v1"
+		(property "Reference" "ev_dcdc_24v"
 			(at 84.328 31.75 0)
 			(effects
@@
 			(project ""
 				(path "/f9355d6c-5335-47ee-824d-8b7223514fe3"
-					(reference "ev_dcdc_24v1")
+					(reference "ev_dcdc_24v")
 					(unit 1)
 				)
@@
 		(on_board yes)
 		(dnp no)
-		(property "Reference" "ev_nucleo2"
+		(property "Reference" "ev_stm32"
 			(at 75.438 109.22 0)
 			(effects
@@
 			(project "AutonomousWiring"
 				(path "/f9355d6c-5335-47ee-824d-8b7223514fe3"
-					(reference "ev_nucleo2")
+					(reference "ev_stm32")
 					(unit 1)
 				)
@@
 		(on_board yes)
 		(dnp no)
-		(property "Reference" "F2"
+		(property "Reference" "F1"
 			(at 46.228 50.8 90)
 			(effects
@@
 			(project "AutonomousWiring"
 				(path "/f9355d6c-5335-47ee-824d-8b7223514fe3"
-					(reference "F2")
+					(reference "F1")
 					(unit 1)
 				)
@@
 		(on_board yes)
 		(dnp no)
-		(property "Reference" "ev_poe_adp1"
+		(property "Reference" "ev_poe_adp"
 			(at 86.36 52.07 0)
 			(effects
@@
 			(project "AutonomousWiring"
 				(path "/f9355d6c-5335-47ee-824d-8b7223514fe3"
-					(reference "ev_poe_adp1")
+					(reference "ev_poe_adp")
 					(unit 1)
 				)
@@
 		(on_board yes)
 		(dnp no)
-		(property "Reference" "ev_dcdc_5v2"
+		(property "Reference" "ev_dcdc_5v"
 			(at 135.636 58.42 0)
 			(effects
@@
 			(project "AutonomousWiring"
 				(path "/f9355d6c-5335-47ee-824d-8b7223514fe3"
-					(reference "ev_dcdc_5v2")
+					(reference "ev_dcdc_5v")
 					(unit 1)
 				)
@@
 		(on_board yes)
 		(dnp no)
-		(property "Reference" "ev_steering2"
+		(property "Reference" "ev_steering"
 			(at 90.424 19.05 0)
 			(effects
@@
 			(project "AutonomousWiring"
 				(path "/f9355d6c-5335-47ee-824d-8b7223514fe3"
-					(reference "ev_steering2")
+					(reference "ev_steering")
 					(unit 1)
 				)
@@
 		(on_board yes)
 		(dnp no)
-		(property "Reference" "ev_battery2"
+		(property "Reference" "ev_battery"
 			(at 22.352 70.866 0)
 			(effects
@@
 			(project "AutonomousWiring"
 				(path "/f9355d6c-5335-47ee-824d-8b7223514fe3"
-					(reference "ev_battery2")
+					(reference "ev_battery")
 					(unit 1)
 				)
@@
 		(on_board yes)
 		(dnp no)
-		(property "Reference" "ev_contactor2"
+		(property "Reference" "ev_contactor"
 			(at 39.116 134.366 0)
 			(effects
@@
 			(project "AutonomousWiring"
 				(path "/f9355d6c-5335-47ee-824d-8b7223514fe3"
-					(reference "ev_contactor2")
+					(reference "ev_contactor")
 					(unit 1)
 				)
@@
 		(on_board yes)
 		(dnp no)
-		(property "Reference" "PreCharge1"
+		(property "Reference" "PreCharge"
 			(at 57.912 50.8 90)
 			(effects
@@
 			(project "AutonomousWiring"
 				(path "/f9355d6c-5335-47ee-824d-8b7223514fe3"
-					(reference "PreCharge1")
+					(reference "PreCharge")
 					(unit 1)
 				)
@@
 		(on_board yes)
 		(dnp no)
-		(property "Reference" "ev_eth_switch1"
+		(property "Reference" "ev_eth_switch"
 			(at 80.01 63.5 0)
 			(effects
@@
 			(project "AutonomousWiring"
 				(path "/f9355d6c-5335-47ee-824d-8b7223514fe3"
-					(reference "ev_eth_switch1")
+					(reference "ev_eth_switch")
 					(unit 1)
 				)
@@
 		(on_board yes)
 		(dnp no)
-		(property "Reference" "ev_rtk_gps1"
+		(property "Reference" "ev_rtk_gps"
 			(at 105.41 96.52 0)
 			(effects
@@
 			(project ""
 				(path "/f9355d6c-5335-47ee-824d-8b7223514fe3"
-					(reference "ev_rtk_gps1")
+					(reference "ev_rtk_gps")
 					(unit 1)
 				)
@@
 		(on_board yes)
 		(dnp no)
-		(property "Reference" "ev_dcusbcpd2"
+		(property "Reference" "ev_dcusbcpd"
 			(at 117.094 60.96 0)
 			(effects
@@
 			(project "AutonomousWiring"
 				(path "/f9355d6c-5335-47ee-824d-8b7223514fe3"
-					(reference "ev_dcusbcpd2")
+					(reference "ev_dcusbcpd")
 					(unit 1)
 				)
@@
 		(on_board yes)
 		(dnp no)
-		(property "Reference" "ev_rc_reciever2"
+		(property "Reference" "ev_rc_reciever"
 			(at 114.3 142.494 0)
 			(effects
@@
 			(project "AutonomousWiring"
 				(path "/f9355d6c-5335-47ee-824d-8b7223514fe3"
-					(reference "ev_rc_reciever2")
+					(reference "ev_rc_reciever")
 					(unit 1)
 				)
@@
 		(on_board yes)
 		(dnp no)
-		(property "Reference" "ev_bullet1"
+		(property "Reference" "ev_bullet"
 			(at 104.14 54.61 0)
 			(effects
@@
 			(project "AutonomousWiring"
 				(path "/f9355d6c-5335-47ee-824d-8b7223514fe3"
-					(reference "ev_bullet1")
+					(reference "ev_bullet")
 					(unit 1)
 				)
@@
 		(on_board yes)
 		(dnp no)
-		(property "Reference" "EStop1"
+		(property "Reference" "EStop"
 			(at 107.95 35.052 0)
 			(effects
@@
 			(project "AutonomousWiring"
 				(path "/f9355d6c-5335-47ee-824d-8b7223514fe3"
-					(reference "EStop1")
+					(reference "EStop")
 					(unit 1)
 				)
@@
 		(on_board yes)
 		(dnp no)
-		(property "Reference" "ev_vesc2"
+		(property "Reference" "ev_vesc"
 			(at 139.954 114.046 0)
 			(effects
@@
 			(project ""
 				(path "/f9355d6c-5335-47ee-824d-8b7223514fe3"
-					(reference "ev_vesc2")
-					(unit 1)
-				)
+					(reference "ev_vesc")
+					(unit 1)
+				)
